File: artProject_X/artProject_X/artProject_X.sch (EAGLE design)
At the start: 29 parts

Commit message: artProjectX stm32
Parts:
- removed JP15, JP16, JP17, JP18, JP19, JP20: (no value), pinhead:PINHD-1X4
- added 5V, GND: (no value), pinhead:PINHD-1X1
- added DECRE, ENTER, INCRE, RESET: (no value), switch-omron:10-XX
- added R1: (no value), resistor:R-EU_0204/7
- added STE1, STE2, STE3, STE4, STE5, STE6: (no value), pinhead:PINHD-1X4
- renumbered JP10 to 3PIN3, JP11 to 3PIN4, JP12 to 3PIN5, JP13 to 3PIN6, JP14 to 3PIN7, JP8 to 3PIN1, JP9 to 3PIN2
Connections:
- new net N$1: 3PIN1.3, 4.33
- new net N$10: 3.6, ENTER.S, ENTER.S1
- new net N$11: 7.3, RESET.S, RESET.S1
- new net N$12: 2.5, STE6.1
- new net N$13: 2.6, STE6.3
- new net N$14: 2.4, STE5.3
- new net N$15: DECRE.P, DECRE.P1, ENTER.P, ENTER.P1, INCRE.P, INCRE.P1, R1.1, RESET.P, RESET.P1
- new net N$16: 2.3, STE5.1
- new net N$17: 2.2, STE4.3
- new net N$18: 2.1, STE4.1
- new net N$19: 1.10, STE3.3
- new net N$20: 1.9, STE3.1
- new net N$21: 1.8, STE2.3
- new net N$22: 1.7, STE2.1
- new net N$23: 1.6, STE1.3
- new net N$24: 1.5, STE1.1
- new net N$3: 3PIN2.3, 4.31
- new net N$5: 3PIN4.3, 4.27
- new net N$6: 3PIN5.3, 4.25
- new net N$7: 3PIN6.3, 4.23
- new net N$8: 3PIN7.3, 4.21
- new net N$9: 3.5, DECRE.S, DECRE.S1
- new net VCC: 3PIN1.2, 3PIN2.2, 3PIN3.2, 3PIN4.2, 3PIN5.2, 3PIN6.2, 3PIN7.2, 4.35, 4.36, 7.5, I2C1.3, I2C2.3, I2C3.3, I2C4.3, I2C5.3, I2C6.3, I2C7.3, I2C8.3, I2CLCD.3, R1.2
- net GND: now also 3PIN1.1, 3PIN2.1, 3PIN3.1, 3PIN4.1, 3PIN5.1, 3PIN6.1, 3PIN7.1, 4.1, 4.2, GND.1, I2C1.4, I2C2.4, I2C3.4, I2C4.4, I2C5.4, I2C6.4, I2C7.4, I2C8.4, I2CLCD.4, STE1.2, STE1.4, STE2.2, STE2.4, STE3.2, STE3.4, STE4.2, STE4.4, STE5.2, STE5.4, STE6.2, STE6.4; no longer 3PIN1.3, 3PIN2.3, 3PIN3.3, 3PIN4.3, 3PIN5.3, 3PIN6.3, 3PIN7.3
- net N$2: now also 3.4, INCRE.S, INCRE.S1; no longer 3PIN1.1, 3PIN2.1, 3PIN3.1, 3PIN4.1, 3PIN5.1, 3PIN6.1, 3PIN7.1, 4.35, 4.36, 7.5, I2C1.1, I2C2.1, I2C3.1, I2C4.1, I2C5.1, I2C6.1, I2C7.1, I2C8.1, I2CLCD.1
- net N$4: now also 3PIN3.3, 4.29; no longer I2C1.4, I2C2.4, I2C3.4, I2C4.4, I2C5.4, I2C6.4, I2C7.4, I2C8.4, I2CLCD.4
- net SCL: now also I2C1.1, I2C2.1, I2C3.1, I2C4.1, I2C5.1, I2C6.1, I2C7.1, I2C8.1, I2CLCD.1; no longer I2C1.3, I2C2.3, I2C3.3, I2C4.3, I2C5.3, I2C6.3, I2C7.3, I2C8.3, I2CLCD.3
