File: artProject_X/artProject_X/artProject_X.brd (EAGLE design)
At the start: 345.4 x 281.6 mm, 29 parts

Commit message: artProjectX stm32
Parts:
- removed JP10, JP11, JP12, JP13, JP14, JP8, JP9: (no value), pinhead:1X03
- removed JP15, JP16, JP17, JP18, JP19, JP20: (no value), pinhead:1X04
- added 3PIN1, 3PIN2, 3PIN3, 3PIN4, 3PIN5, 3PIN6, 3PIN7: (no value), pinhead:1X03
- added 5V, GND: (no value), pinhead:1X01
- added DECRE, ENTER, INCRE, RESET: (no value), switch-omron:B3F-10XX
- added R1: (no value), resistor:0204/7
- added STE1, STE2, STE3, STE4, STE5, STE6: (no value), pinhead:1X04
- moved I2CLCD 198.0 mm to (-29.2, 167.6)
- moved 1 84.3 mm to (-30.5, 49.5)
- moved 2 84.3 mm to (-5.08, 49.5)
- moved 3 84.3 mm to (17.8, 49.5)
- moved 5 84.3 mm to (17.8, 1.27)
- moved 6 84.3 mm to (-5.08, 1.27)
- moved 7 84.3 mm to (-27.9, 1.27)
- moved 4 84.3 mm to (34.3, 26.7)
- moved I2C4 54.0 mm to (116.8, 118.1), turned to 0 degrees
- moved I2C6 54.0 mm to (116.8, 87.6), turned to 0 degrees
- moved I2C1 54.0 mm to (116.8, 163.8), turned to 0 degrees
- moved I2C2 54.0 mm to (116.8, 148.6), turned to 0 degrees
- moved I2C3 54.0 mm to (116.8, 133.3), turned to 0 degrees
- moved I2C5 54.0 mm to (116.8, 102.9), turned to 0 degrees
- moved I2C7 54.0 mm to (116.8, 72.4), turned to 0 degrees
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Connections:
- new net N$1: 3PIN1.3, 4.33
- new net N$10: 3.6, ENTER.1, ENTER.2
- new net N$11: 7.3, RESET.1, RESET.2
- new net N$12: 2.5, STE6.1
- new net N$13: 2.6, STE6.3
- new net N$14: 2.4, STE5.3
- new net N$15: DECRE.3, DECRE.4, ENTER.3, ENTER.4, INCRE.3, INCRE.4, R1.1, RESET.3, RESET.4
- new net N$16: 2.3, STE5.1
- new net N$17: 2.2, STE4.3
- new net N$18: 2.1, STE4.1
- new net N$19: 1.10, STE3.3
- new net N$20: 1.9, STE3.1
- new net N$21: 1.8, STE2.3
- new net N$22: 1.7, STE2.1
- new net N$23: 1.6, STE1.3
- new net N$24: 1.5, STE1.1
- new net N$3: 3PIN2.3, 4.31
- new net N$5: 3PIN4.3, 4.27
- new net N$6: 3PIN5.3, 4.25
- new net N$7: 3PIN6.3, 4.23
- new net N$8: 3PIN7.3, 4.21
- new net N$9: 3.5, DECRE.1, DECRE.2
- new net VCC: 3PIN1.2, 3PIN2.2, 3PIN3.2, 3PIN4.2, 3PIN5.2, 3PIN6.2, 3PIN7.2, 4.35, 4.36, 7.5, I2C1.3, I2C2.3, I2C3.3, I2C4.3, I2C5.3, I2C6.3, I2C7.3, I2C8.3, I2CLCD.3, R1.2
- net GND: now also 3PIN1.1, 3PIN2.1, 3PIN3.1, 3PIN4.1, 3PIN5.1, 3PIN6.1, 3PIN7.1, 4.1, 4.2, GND.1, I2C1.4, I2C2.4, I2C3.4, I2C4.4, I2C5.4, I2C6.4, I2C7.4, I2C8.4, I2CLCD.4, STE1.2, STE1.4, STE2.2, STE2.4, STE3.2, STE3.4, STE4.2, STE4.4, STE5.2, STE5.4, STE6.2, STE6.4; no longer JP10.3, JP11.3, JP12.3, JP13.3, JP14.3, JP8.3, JP9.3
- net N$2: now also 3.4, INCRE.1, INCRE.2; no longer 4.35, 4.36, 7.5, I2C1.1, I2C2.1, I2C3.1, I2C4.1, I2C5.1, I2C6.1, I2C7.1, I2C8.1, I2CLCD.1, JP10.1, JP11.1, JP12.1, JP13.1, JP14.1, JP8.1, JP9.1
- net N$4: now also 3PIN3.3, 4.29; no longer I2C1.4, I2C2.4, I2C3.4, I2C4.4, I2C5.4, I2C6.4, I2C7.4, I2C8.4, I2CLCD.4
- net SCL: now also I2C1.1, I2C2.1, I2C3.1, I2C4.1, I2C5.1, I2C6.1, I2C7.1, I2C8.1, I2CLCD.1; no longer I2C1.3, I2C2.3, I2C3.3, I2C4.3, I2C5.3, I2C6.3, I2C7.3, I2C8.3, I2CLCD.3
Routing:
- net VCC: track 0.00 -> 648.7 mm
- net N$11: track 0.00 -> 179.1 mm
- net N$2: track 253.1 -> 101.0 mm, vias 4 -> 0
- net N$8: track 0.00 -> 108.7 mm
- net N$7: track 0.00 -> 102.4 mm
- net N$10: track 0.00 -> 101.0 mm
- net N$6: track 0.00 -> 96.8 mm
- net N$9: track 0.00 -> 95.7 mm
- net N$5: track 0.00 -> 91.0 mm
- net N$4: track 0.00 -> 86.7 mm
- net N$3: track 0.00 -> 79.6 mm
- net N$1: track 0.00 -> 77.5 mm
- net SDA: track 295.2 -> 354.5 mm
- net N$15: track 0.00 -> 39.5 mm
- net SCL: track 307.2 -> 342.9 mm, vias 0 -> 2
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- added copper zone on layer 16, net GND

Commit message: stm board complete files
Parts:
- moved STE1 90.6 mm to (-36.8, 69.8)
- moved STE2 87.6 mm to (-27.9, 62.2)
- moved STE6 77.7 mm to (5.08, 62.2)
- moved STE5 75.9 mm to (1.27, 69.8)
- moved STE4 75.2 mm to (-11.4, 62.2)
- moved STE3 74.5 mm to (-19.1, 69.8)
Changed lines of the file:
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@@
 <element name="3PIN6" library="pinhead" library_urn="urn:adsk.eagle:library:325" package="1X03" package3d_urn="urn:adsk.eagle:package:22458/2" value="" x="115.57" y="5.08" rot="R180"/>
 <element name="3PIN7" library="pinhead" library_urn="urn:adsk.eagle:library:325" package="1X03" package3d_urn="urn:adsk.eagle:package:22458/2" value="" x="115.57" y="-3.81" rot="R180"/>
-<element name="STE1" library="pinhead" library_urn="urn:adsk.eagle:library:325" package="1X04" package3d_urn="urn:adsk.eagle:package:22407/2" value="" x="-71.12" y="153.67"/>
-<element name="STE2" library="pinhead" library_urn="urn:adsk.eagle:library:325" package="1X04" package3d_urn="urn:adsk.eagle:package:22407/2" value="" x="-71.12" y="138.43"/>
-<element name="STE3" library="pinhead" library_urn="urn:adsk.eagle:library:325" package="1X04" package3d_urn="urn:adsk.eagle:package:22407/2" value="" x="-71.12" y="123.19"/>
-<element name="STE4" library="pinhead" library_urn="urn:adsk.eagle:library:325" package="1X04" package3d_urn="urn:adsk.eagle:package:22407/2" value="" x="-71.12" y="107.95"/>
-<element name="STE5" library="pinhead" library_urn="urn:adsk.eagle:library:325" package="1X04" package3d_urn="urn:adsk.eagle:package:22407/2" value="" x="-71.12" y="92.71"/>
-<element name="STE6" library="pinhead" library_urn="urn:adsk.eagle:library:325" package="1X04" package3d_urn="urn:adsk.eagle:package:22407/2" value="" x="-71.12" y="77.47"/>
+<element name="STE1" library="pinhead" library_urn="urn:adsk.eagle:library:325" package="1X04" package3d_urn="urn:adsk.eagle:package:22407/2" value="" x="-36.83" y="69.85"/>
+<element name="STE2" library="pinhead" library_urn="urn:adsk.eagle:library:325" package="1X04" package3d_urn="urn:adsk.eagle:package:22407/2" value="" x="-27.94" y="62.23"/>
+<element name="STE3" library="pinhead" library_urn="urn:adsk.eagle:library:325" package="1X04" package3d_urn="urn:adsk.eagle:package:22407/2" value="" x="-19.05" y="69.85"/>
+<element name="STE4" library="pinhead" library_urn="urn:adsk.eagle:library:325" package="1X04" package3d_urn="urn:adsk.eagle:package:22407/2" value="" x="-11.43" y="62.23"/>
+<element name="STE5" library="pinhead" library_urn="urn:adsk.eagle:library:325" package="1X04" package3d_urn="urn:adsk.eagle:package:22407/2" value="" x="1.27" y="69.85"/>
+<element name="STE6" library="pinhead" library_urn="urn:adsk.eagle:library:325" package="1X04" package3d_urn="urn:adsk.eagle:package:22407/2" value="" x="5.08" y="62.23"/>
 <element name="I2C1" library="pinhead" library_urn="urn:adsk.eagle:library:325" package="1X04" package3d_urn="urn:adsk.eagle:package:22407/2" value="" x="116.84" y="163.83"/>
 <element name="I2C2" library="pinhead" library_urn="urn:adsk.eagle:library:325" package="1X04" package3d_urn="urn:adsk.eagle:package:22407/2" value="" x="116.84" y="148.59"/>
@@
 <contactref element="STE5" pad="4"/>
 <contactref element="STE6" pad="2"/>
-<wire x1="120.65" y1="118.11" x2="120.65" y2="133.35" width="0" layer="19" extent="1-1"/>
-<wire x1="120.65" y1="102.87" x2="120.65" y2="118.11" width="0" layer="19" extent="1-1"/>
-<wire x1="120.65" y1="87.63" x2="120.65" y2="102.87" width="0" layer="19" extent="1-1"/>
-<wire x1="120.65" y1="72.39" x2="120.65" y2="87.63" width="0" layer="19" extent="1-1"/>
-<wire x1="120.65" y1="57.15" x2="120.65" y2="72.39" width="0" layer="19" extent="1-1"/>
-<wire x1="118.11" y1="45.72" x2="120.65" y2="57.15" width="0" layer="19" extent="1-1"/>
-<wire x1="118.11" y1="38.1" x2="118.11" y2="45.72" width="0" layer="19" extent="1-1"/>
-<wire x1="118.11" y1="29.21" x2="118.11" y2="38.1" width="0" layer="19" extent="1-1"/>
-<wire x1="118.11" y1="21.59" x2="118.11" y2="29.21" width="0" layer="19" extent="1-1"/>
-<wire x1="118.11" y1="13.97" x2="118.11" y2="21.59" width="0" layer="19" extent="1-1"/>
-<wire x1="118.11" y1="5.08" x2="118.11" y2="13.97" width="0" layer="19" extent="1-1"/>
-<wire x1="118.11" y1="-3.81" x2="118.11" y2="5.08" width="0" layer="19" extent="1-1"/>
-<wire x1="120.65" y1="148.59" x2="120.65" y2="133.35" width="0" layer="19" extent="1-1"/>
-<wire x1="120.65" y1="163.83" x2="120.65" y2="148.59" width="0" layer="19" extent="1-1"/>
-<wire x1="35.56" y1="5.08" x2="118.11" y2="5.08" width="0" layer="19" extent="1-1"/>
-<wire x1="33.02" y1="5.08" x2="35.56" y2="5.08" width="0" layer="19" extent="1-1"/>
-<wire x1="-21.59" y1="1.27" x2="33.02" y2="5.08" width="0" layer="19" extent="1-1"/>
-<wire x1="-67.31" y1="77.47" x2="-24.13" y2="1.27" width="0" layer="19" extent="1-1"/>
-<wire x1="-72.39" y1="77.47" x2="-67.31" y2="77.47" width="0" layer="19" extent="1-1"/>
-<wire x1="-67.31" y1="92.71" x2="-67.31" y2="77.47" width="0" layer="19" extent="1-1"/>
-<wire x1="-72.39" y1="92.71" x2="-67.31" y2="92.71" width="0" layer="19" extent="1-1"/>
-<wire x1="-67.31" y1="107.95" x2="-67.31" y2="92.71" width="0" layer="19" extent="1-1"/>
-<wire x1="-72.39" y1="107.95" x2="-67.31" y2="107.95" width="0" layer="19" extent="1-1"/>
-<wire x1="-67.31" y1="123.19" x2="-67.31" y2="107.95" width="0" layer="19" extent="1-1"/>
-<wire x1="-72.39" y1="123.19" x2="-67.31" y2="123.19" width="0" layer="19" extent="1-1"/>
-<wire x1="-67.31" y1="138.43" x2="-67.31" y2="123.19" width="0" layer="19" extent="1-1"/>
-<wire x1="-72.39" y1="138.43" x2="-67.31" y2="138.43" width="0" layer="19" extent="1-1"/>
-<wire x1="-67.31" y1="153.67" x2="-67.31" y2="138.43" width="0" layer="19" extent="1-1"/>
-<wire x1="-72.39" y1="153.67" x2="-67.31" y2="153.67" width="0" layer="19" extent="1-1"/>
-<wire x1="-29.21" y1="171.45" x2="-67.31" y2="107.95" width="0" layer="19" extent="1-1"/>
-<wire x1="-72.39" y1="200.66" x2="-72.39" y2="153.67" width="0" layer="19" extent="1-1"/>
 </signal>
 <signal name="N$1">
@@
 <contactref element="STE6" pad="1"/>
 <contactref element="2" pad="5"/>
-<wire x1="-74.93" y1="77.47" x2="-3.81" y2="49.53" width="0" layer="19" extent="1-1"/>
+<wire x1="1.27" y1="62.23" x2="-3.81" y2="49.53" width="0" layer="19" extent="1-1"/>
 </signal>
 <signal name="N$13">
 <contactref element="2" pad="6"/>
 <contactref element="STE6" pad="3"/>
-<wire x1="-69.85" y1="77.47" x2="-1.27" y2="49.53" width="0" layer="19" extent="1-1"/>
+<wire x1="6.35" y1="62.23" x2="-1.27" y2="49.53" width="0" layer="19" extent="1-1"/>
 </signal>
 <signal name="N$14">
 <contactref element="STE5" pad="3"/>
 <contactref element="2" pad="4"/>
-<wire x1="-69.85" y1="92.71" x2="-6.35" y2="49.53" width="0" layer="19" extent="1-1"/>
+<wire x1="2.54" y1="69.85" x2="-6.35" y2="49.53" width="0" layer="19" extent="1-1"/>
 </signal>
 <signal name="N$16">
 <contactref element="2" pad="3"/>
 <contactref element="STE5" pad="1"/>
-<wire x1="-74.93" y1="92.71" x2="-8.89" y2="49.53" width="0" layer="19" extent="1-1"/>
+<wire x1="-2.54" y1="69.85" x2="-8.89" y2="49.53" width="0" layer="19" extent="1-1"/>
 </signal>
 <signal name="N$17">
 <contactref element="STE4" pad="3"/>
 <contactref element="2" pad="2"/>
-<wire x1="-11.43" y1="49.53" x2="-69.85" y2="107.95" width="0" layer="19" extent="1-1"/>
+<wire x1="-11.43" y1="49.53" x2="-10.16" y2="62.23" width="0" layer="19" extent="1-1"/>
 </signal>
 <signal name="N$18">
 <contactref element="2" pad="1"/>
 <contactref element="STE4" pad="1"/>
-<wire x1="-74.93" y1="107.95" x2="-13.97" y2="49.53" width="0" layer="19" extent="1-1"/>
+<wire x1="-15.24" y1="62.23" x2="-13.97" y2="49.53" width="0" layer="19" extent="1-1"/>
 </signal>
 <signal name="N$19">
 <contactref element="STE3" pad="3"/>
 <contactref element="1" pad="10"/>
-<wire x1="-19.05" y1="49.53" x2="-69.85" y2="123.19" width="0" layer="19" extent="1-1"/>
+<wire x1="-19.05" y1="49.53" x2="-17.78" y2="69.85" width="0" layer="19" extent="1-1"/>
 </signal>
 <signal name="N$20">
 <contactref element="STE3" pad="1"/>
 <contactref element="1" pad="9"/>
-<wire x1="-21.59" y1="49.53" x2="-74.93" y2="123.19" width="0" layer="19" extent="1-1"/>
+<wire x1="-21.59" y1="49.53" x2="-22.86" y2="69.85" width="0" layer="19" extent="1-1"/>
 </signal>
 <signal name="N$21">
 <contactref element="STE2" pad="3"/>
 <contactref element="1" pad="8"/>
-<wire x1="-24.13" y1="49.53" x2="-69.85" y2="138.43" width="0" layer="19" extent="1-1"/>
+<wire x1="-24.13" y1="49.53" x2="-26.67" y2="62.23" width="0" layer="19" extent="1-1"/>
 </signal>
 <signal name="N$22">
 <contactref element="1" pad="7"/>
 <contactref element="STE2" pad="1"/>
-<wire x1="-26.67" y1="49.53" x2="-74.93" y2="138.43" width="0" layer="19" extent="1-1"/>
+<wire x1="-26.67" y1="49.53" x2="-31.75" y2="62.23" width="0" layer="19" extent="1-1"/>
 </signal>
 <signal name="N$23">
 <contactref element="STE1" pad="3"/>
 <contactref element="1" pad="6"/>
-<wire x1="-29.21" y1="49.53" x2="-69.85" y2="153.67" width="0" layer="19" extent="1-1"/>
+<wire x1="-29.21" y1="49.53" x2="-35.56" y2="69.85" width="0" layer="19" extent="1-1"/>
 </signal>
 <signal name="N$24">
 <contactref element="1" pad="5"/>
 <contactref element="STE1" pad="1"/>
-<wire x1="-31.75" y1="49.53" x2="-74.93" y2="153.67" width="0" layer="19" extent="1-1"/>
+<wire x1="-31.75" y1="49.53" x2="-40.64" y2="69.85" width="0" layer="19" extent="1-1"/>
 </signal>
 </signals>

Commit message: servo code
Routing:
- net N$14: track 0.00 -> 24.6 mm
- net N$24: track 0.00 -> 23.9 mm
- net N$23: track 0.00 -> 22.9 mm
- net N$16: track 0.00 -> 22.8 mm
- net N$20: track 0.00 -> 20.8 mm
- net N$19: track 0.00 -> 20.8 mm
- net N$13: track 0.00 -> 17.2 mm
- net N$22: track 0.00 -> 14.7 mm
- net N$12: track 0.00 -> 14.7 mm
- net N$21: track 0.00 -> 13.7 mm
- net N$18: track 0.00 -> 13.2 mm
- net N$17: track 0.00 -> 13.2 mm
Changed lines of the file:
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@@
 <contactref element="STE5" pad="4"/>
 <contactref element="STE6" pad="2"/>
+<wire x1="-24.13" y1="62.23" x2="-29.21" y2="62.23" width="0" layer="19" extent="1-1"/>
 </signal>
 <signal name="N$1">
@@
 <contactref element="STE6" pad="1"/>
 <contactref element="2" pad="5"/>
-<wire x1="1.27" y1="62.23" x2="-3.81" y2="49.53" width="0" layer="19" extent="1-1"/>
+<wire x1="-3.81" y1="49.53" x2="-3.81" y2="51.6557875" width="0.8128" layer="16"/>
+<wire x1="-3.81" y1="51.6557875" x2="-3.51710625" y2="52.36289375" width="0.8128" layer="16" curve="-45"/>
+<wire x1="0.97710625" y1="56.85710625" x2="1.27" y2="57.5642125" width="0.8128" layer="16" curve="45"/>
+<wire x1="1.27" y1="57.5642125" x2="1.27" y2="62.23" width="0.8128" layer="16"/>
+<wire x1="-3.51710625" y1="52.36289375" x2="0.97710625" y2="56.85710625" width="0.8128" layer="16"/>
 </signal>
 <signal name="N$13">
 <contactref element="2" pad="6"/>
 <contactref element="STE6" pad="3"/>
-<wire x1="6.35" y1="62.23" x2="-1.27" y2="49.53" width="0" layer="19" extent="1-1"/>
+<wire x1="6.35" y1="62.23" x2="6.35" y2="57.15" width="0.8128" layer="16"/>
+<wire x1="6.35" y1="57.15" x2="5.37289375" y2="56.17289375" width="0.8128" layer="16"/>
+<wire x1="5.37289375" y1="56.17289375" x2="4.6657875" y2="55.88" width="0.8128" layer="16" curve="-45"/>
+<wire x1="2.9542125" y1="55.88" x2="2.24710625" y2="55.58710625" width="0.8128" layer="16" curve="45"/>
+<wire x1="2.24710625" y1="55.58710625" x2="-1.27" y2="52.07" width="0.8128" layer="16"/>
+<wire x1="-1.27" y1="52.07" x2="-1.27" y2="49.53" width="0.8128" layer="16"/>
+<wire x1="4.6657875" y1="55.88" x2="2.9542125" y2="55.88" width="0.8128" layer="16"/>
 </signal>
 <signal name="N$14">
 <contactref element="STE5" pad="3"/>
 <contactref element="2" pad="4"/>
-<wire x1="2.54" y1="69.85" x2="-6.35" y2="49.53" width="0" layer="19" extent="1-1"/>
+<wire x1="2.54" y1="69.85" x2="2.54" y2="67.31" width="0.8128" layer="16"/>
+<wire x1="2.54" y1="67.31" x2="1.56289375" y2="66.33289375" width="0.8128" layer="16"/>
+<wire x1="1.56289375" y1="66.33289375" x2="0.8557875" y2="66.04" width="0.8128" layer="16" curve="-45"/>
+<wire x1="0.8557875" y1="66.04" x2="0" y2="66.04" width="0.8128" layer="16"/>
+<wire x1="0" y1="66.04" x2="-2.54" y2="63.5" width="0.8128" layer="16"/>
+<wire x1="-2.54" y1="56.2942125" x2="-2.83289375" y2="55.58710625" width="0.8128" layer="16" curve="-45"/>
+<wire x1="-2.83289375" y1="55.58710625" x2="-6.35" y2="52.07" width="0.8128" layer="16"/>
+<wire x1="-6.35" y1="52.07" x2="-6.35" y2="49.53" width="0.8128" layer="16"/>
+<wire x1="-2.54" y1="63.5" x2="-2.54" y2="56.2942125" width="0.8128" layer="16"/>
 </signal>
 <signal name="N$16">
 <contactref element="2" pad="3"/>
 <contactref element="STE5" pad="1"/>
-<wire x1="-2.54" y1="69.85" x2="-8.89" y2="49.53" width="0" layer="19" extent="1-1"/>
+<wire x1="-8.89" y1="49.53" x2="-8.89" y2="52.9257875" width="0.8128" layer="16"/>
+<wire x1="-8.89" y1="52.9257875" x2="-8.59710625" y2="53.63289375" width="0.8128" layer="16" curve="-45"/>
+<wire x1="-8.59710625" y1="53.63289375" x2="-5.08" y2="57.15" width="0.8128" layer="16"/>
+<wire x1="-5.08" y1="57.15" x2="-5.08" y2="63.0857875" width="0.8128" layer="16"/>
+<wire x1="-5.08" y1="63.0857875" x2="-4.78710625" y2="63.79289375" width="0.8128" layer="16" curve="-45"/>
+<wire x1="-4.78710625" y1="63.79289375" x2="-2.54" y2="66.04" width="0.8128" layer="16"/>
+<wire x1="-2.54" y1="66.04" x2="-2.54" y2="69.85" width="0.8128" layer="16"/>
 </signal>
 <signal name="N$17">
 <contactref element="STE4" pad="3"/>
 <contactref element="2" pad="2"/>
-<wire x1="-11.43" y1="49.53" x2="-10.16" y2="62.23" width="0" layer="19" extent="1-1"/>
+<wire x1="-10.16" y1="62.23" x2="-10.16" y2="57.5642125" width="0.8128" layer="16"/>
+<wire x1="-10.16" y1="57.5642125" x2="-10.45289375" y2="56.85710625" width="0.8128" layer="16" curve="-45"/>
+<wire x1="-10.45289375" y1="56.85710625" x2="-11.43" y2="55.88" width="0.8128" layer="16"/>
+<wire x1="-11.43" y1="55.88" x2="-11.43" y2="49.53" width="0.8128" layer="16"/>
 </signal>
 <signal name="N$18">
 <contactref element="2" pad="1"/>
 <contactref element="STE4" pad="1"/>
-<wire x1="-15.24" y1="62.23" x2="-13.97" y2="49.53" width="0" layer="19" extent="1-1"/>
+<wire x1="-15.24" y1="62.23" x2="-15.24" y2="57.5642125" width="0.8128" layer="16"/>
+<wire x1="-15.24" y1="57.5642125" x2="-14.94710625" y2="56.85710625" width="0.8128" layer="16" curve="45"/>
+<wire x1="-14.94710625" y1="56.85710625" x2="-13.97" y2="55.88" width="0.8128" layer="16"/>
+<wire x1="-13.97" y1="55.88" x2="-13.97" y2="49.53" width="0.8128" layer="16"/>
 </signal>
 <signal name="N$19">
 <contactref element="STE3" pad="3"/>
 <contactref element="1" pad="10"/>
-<wire x1="-19.05" y1="49.53" x2="-17.78" y2="69.85" width="0" layer="19" extent="1-1"/>
+<wire x1="-17.78" y1="69.85" x2="-17.78" y2="66.4542125" width="0.8128" layer="16"/>
+<wire x1="-17.78" y1="66.4542125" x2="-18.07289375" y2="65.74710625" width="0.8128" layer="16" curve="-45"/>
+<wire x1="-18.07289375" y1="65.74710625" x2="-19.05" y2="64.77" width="0.8128" layer="16"/>
+<wire x1="-19.05" y1="64.77" x2="-19.05" y2="49.53" width="0.8128" layer="16"/>
 </signal>
 <signal name="N$20">
 <contactref element="STE3" pad="1"/>
 <contactref element="1" pad="9"/>
-<wire x1="-21.59" y1="49.53" x2="-22.86" y2="69.85" width="0" layer="19" extent="1-1"/>
+<wire x1="-21.59" y1="49.53" x2="-21.59" y2="64.3557875" width="0.8128" layer="16"/>
+<wire x1="-21.59" y1="64.3557875" x2="-21.88289375" y2="65.06289375" width="0.8128" layer="16" curve="45"/>
+<wire x1="-21.88289375" y1="65.06289375" x2="-22.86" y2="66.04" width="0.8128" layer="16"/>
+<wire x1="-22.86" y1="66.04" x2="-22.86" y2="69.85" width="0.8128" layer="16"/>
 </signal>
 <signal name="N$21">
 <contactref element="STE2" pad="3"/>
 <contactref element="1" pad="8"/>
-<wire x1="-24.13" y1="49.53" x2="-26.67" y2="62.23" width="0" layer="19" extent="1-1"/>
+<wire x1="-26.67" y1="62.23" x2="-26.67" y2="58.42" width="0.8128" layer="16"/>
+<wire x1="-26.67" y1="58.42" x2="-24.42289375" y2="56.17289375" width="0.8128" layer="16"/>
+<wire x1="-24.42289375" y1="56.17289375" x2="-24.13" y2="55.4657875" width="0.8128" layer="16" curve="-45"/>
+<wire x1="-24.13" y1="55.4657875" x2="-24.13" y2="49.53" width="0.8128" layer="16"/>
 </signal>
 <signal name="N$22">
 <contactref element="1" pad="7"/>
 <contactref element="STE2" pad="1"/>
-<wire x1="-26.67" y1="49.53" x2="-31.75" y2="62.23" width="0" layer="19" extent="1-1"/>
+<wire x1="-31.75" y1="62.23" x2="-31.75" y2="60.1042125" width="0.8128" layer="16"/>
+<wire x1="-31.75" y1="60.1042125" x2="-31.45710625" y2="59.39710625" width="0.8128" layer="16" curve="45"/>
+<wire x1="-31.45710625" y1="59.39710625" x2="-26.67" y2="54.61" width="0.8128" layer="16"/>
+<wire x1="-26.67" y1="54.61" x2="-26.67" y2="49.53" width="0.8128" layer="16"/>
 </signal>
 <signal name="N$23">
 <contactref element="STE1" pad="3"/>
 <contactref element="1" pad="6"/>
-<wire x1="-29.21" y1="49.53" x2="-35.56" y2="69.85" width="0" layer="19" extent="1-1"/>
+<wire x1="-35.56" y1="69.85" x2="-35.56" y2="61.3742125" width="0.8128" layer="16"/>
+<wire x1="-35.56" y1="61.3742125" x2="-35.26710625" y2="60.66710625" width="0.8128" layer="16" curve="45"/>
+<wire x1="-35.26710625" y1="60.66710625" x2="-29.21" y2="54.61" width="0.8128" layer="16"/>
+<wire x1="-29.21" y1="54.61" x2="-29.21" y2="49.53" width="0.8128" layer="16"/>
 </signal>
 <signal name="N$24">
 <contactref element="1" pad="5"/>
 <contactref element="STE1" pad="1"/>
-<wire x1="-31.75" y1="49.53" x2="-40.64" y2="69.85" width="0" layer="19" extent="1-1"/>
+<wire x1="-31.75" y1="49.53" x2="-31.75" y2="53.34" width="0.8128" layer="16"/>
+<wire x1="-31.75" y1="53.34" x2="-40.34710625" y2="61.93710625" width="0.8128" layer="16"/>
+<wire x1="-40.34710625" y1="61.93710625" x2="-40.64" y2="62.6442125" width="0.8128" layer="16" curve="-45"/>
+<wire x1="-40.64" y1="62.6442125" x2="-40.64" y2="69.85" width="0.8128" layer="16"/>
 </signal>
 </signals>
