File: Repo_PCB/LSA/LSA.brd (EAGLE design)
At the start: 160 x 100 mm, 5 parts

Commit message: Gerber files
Changed lines of the file:
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@@
 <?xml version="1.0" encoding="utf-8"?>
 <!DOCTYPE eagle SYSTEM "eagle.dtd">
-<eagle version="8.5.2">
+<eagle version="9.2.1">
 <drawing>
 <settings>
@@
 <layer number="14" name="Route14" color="1" fill="6" visible="no" active="no"/>
 <layer number="15" name="Route15" color="4" fill="6" visible="no" active="no"/>
-<layer number="16" name="Bottom" color="15" fill="1" visible="yes" active="yes"/>
+<layer number="16" name="Bottom" color="1" fill="1" visible="yes" active="yes"/>
 <layer number="17" name="Pads" color="15" fill="1" visible="yes" active="yes"/>
 <layer number="18" name="Vias" color="2" fill="1" visible="yes" active="yes"/>
-<layer number="19" name="Unrouted" color="6" fill="1" visible="no" active="yes"/>
+<layer number="19" name="Unrouted" color="6" fill="1" visible="yes" active="yes"/>
 <layer number="20" name="Dimension" color="24" fill="1" visible="no" active="yes"/>
 <layer number="21" name="tPlace" color="7" fill="1" visible="no" active="yes"/>
@@
 <param name="checkStop" value="0"/>
 <param name="checkValues" value="0"/>
+<param name="checkNames" value="1"/>
+<param name="checkWireStubs" value="1"/>
+<param name="checkPolygonWidth" value="0"/>
 <param name="useDiameter" value="13"/>
 <param name="maxErrors" value="50"/>
@@
 </autorouter>
 <elements>
-<element name="JP1" library="pinhead" library_urn="urn:adsk.eagle:library:325" package="2X05" package3d_urn="urn:adsk.eagle:package:22470/2" value="" x="69.85" y="49.53" rot="R270"/>
-<element name="JP2" library="pinhead" library_urn="urn:adsk.eagle:library:325" package="2X05" package3d_urn="urn:adsk.eagle:package:22470/2" value="" x="82.55" y="49.53" rot="R270"/>
-<element name="JP3" library="pinhead" library_urn="urn:adsk.eagle:library:325" package="2X05" package3d_urn="urn:adsk.eagle:package:22470/2" value="" x="95.25" y="49.53" rot="R270"/>
-<element name="VCC" library="pinhead" library_urn="urn:adsk.eagle:library:325" package="1X01" package3d_urn="urn:adsk.eagle:package:22485/2" value="" x="77.47" y="63.5"/>
-<element name="GND" library="pinhead" library_urn="urn:adsk.eagle:library:325" package="1X01" package3d_urn="urn:adsk.eagle:package:22485/2" value="" x="82.55" y="63.5"/>
+<element name="JP1" library="pinhead" library_urn="urn:adsk.eagle:library:325" package="2X05" package3d_urn="urn:adsk.eagle:package:22470/2" value="" x="69.85" y="49.53" smashed="yes" rot="R270">
+<attribute name="NAME" x="73.025" y="55.88" size="1.27" layer="25" ratio="10" rot="R270"/>
+<attribute name="VALUE" x="65.405" y="55.88" size="1.27" layer="27" rot="R270"/>
+</element>
+<element name="JP2" library="pinhead" library_urn="urn:adsk.eagle:library:325" package="2X05" package3d_urn="urn:adsk.eagle:package:22470/2" value="" x="82.55" y="49.53" smashed="yes" rot="R270">
+<attribute name="NAME" x="85.725" y="55.88" size="1.27" layer="25" ratio="10" rot="R270"/>
+<attribute name="VALUE" x="78.105" y="55.88" size="1.27" layer="27" rot="R270"/>
+</element>
+<element name="JP3" library="pinhead" library_urn="urn:adsk.eagle:library:325" package="2X05" package3d_urn="urn:adsk.eagle:package:22470/2" value="" x="95.25" y="49.53" smashed="yes" rot="R270">
+<attribute name="NAME" x="98.425" y="55.88" size="1.27" layer="25" ratio="10" rot="R270"/>
+<attribute name="VALUE" x="90.805" y="55.88" size="1.27" layer="27" rot="R270"/>
+</element>
+<element name="VCC" library="pinhead" library_urn="urn:adsk.eagle:library:325" package="1X01" package3d_urn="urn:adsk.eagle:package:22485/2" value="" x="77.47" y="63.5" smashed="yes">
+<attribute name="NAME" x="76.1238" y="65.3288" size="1.27" layer="25" ratio="10"/>
+<attribute name="VALUE" x="76.2" y="60.325" size="1.27" layer="27"/>
+</element>
+<element name="GND" library="pinhead" library_urn="urn:adsk.eagle:library:325" package="1X01" package3d_urn="urn:adsk.eagle:package:22485/2" value="" x="82.55" y="63.5" smashed="yes">
+<attribute name="NAME" x="81.2038" y="65.3288" size="1.27" layer="25" ratio="10"/>
+<attribute name="VALUE" x="81.28" y="60.325" size="1.27" layer="27"/>
+</element>
 </elements>
 <signals>
@@
 <contactref element="JP1" pad="10"/>
 <contactref element="JP3" pad="10"/>
-<wire x1="71.12" y1="44.45" x2="76.2" y2="44.45" width="0" layer="19" extent="1-16"/>
 <via x="76.2" y="44.45" extent="1-16" drill="0.35"/>
 <wire x1="76.2" y1="44.45" x2="74.93" y2="41.91" width="0.508" layer="1"/>
 <via x="64.77" y="40.64" extent="1-16" drill="0.35"/>
-<wire x1="64.77" y1="40.64" x2="60.96" y2="44.45" width="0" layer="19" extent="1-16"/>
-<wire x1="60.96" y1="44.45" x2="60.96" y2="63.5" width="0" layer="19" extent="1-16"/>
-<wire x1="60.96" y1="63.5" x2="63.5" y2="66.04" width="0" layer="19" extent="1-16"/>
-<wire x1="80.01" y1="66.04" x2="82.55" y2="63.5" width="0" layer="19" extent="1-16"/>
 <wire x1="74.93" y1="41.91" x2="64.77" y2="40.64" width="0.508" layer="1"/>
-<wire x1="63.5" y1="66.04" x2="80.01" y2="66.04" width="0" layer="19" extent="1-16"/>
 </signal>
 <signal name="N$3">
@@
 </signal>
 </signals>
+<mfgpreviewcolors>
+<mfgpreviewcolor name="soldermaskcolor" color="0xC8008000"/>
+<mfgpreviewcolor name="silkscreencolor" color="0xFFFEFEFE"/>
+<mfgpreviewcolor name="backgroundcolor" color="0xFF282828"/>
+<mfgpreviewcolor name="coppercolor" color="0xFFFFBF00"/>
+<mfgpreviewcolor name="substratecolor" color="0xFF786E46"/>
+</mfgpreviewcolors>
 </board>
 </drawing>
