File: Repo_PCB/LSM_PCB/tejesh.brd (EAGLE design)
At the start: 77.5 x 63.2 mm, 6 parts

Commit message: Gerber files
Changed lines of the file:
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@@
 <?xml version="1.0" encoding="utf-8"?>
 <!DOCTYPE eagle SYSTEM "eagle.dtd">
-<eagle version="8.6.0">
+<eagle version="9.2.1">
 <drawing>
 <settings>
@@
 <layer number="14" name="Route14" color="22" fill="1" visible="no" active="no"/>
 <layer number="15" name="Route15" color="23" fill="1" visible="no" active="no"/>
-<layer number="16" name="Bottom" color="1" fill="1" visible="no" active="yes"/>
+<layer number="16" name="Bottom" color="1" fill="1" visible="yes" active="yes"/>
 <layer number="17" name="Pads" color="15" fill="1" visible="yes" active="yes"/>
 <layer number="18" name="Vias" color="15" fill="1" visible="yes" active="yes"/>
@@
 <param name="checkStop" value="0"/>
 <param name="checkValues" value="0"/>
+<param name="checkNames" value="1"/>
+<param name="checkWireStubs" value="1"/>
+<param name="checkPolygonWidth" value="0"/>
 <param name="useDiameter" value="13"/>
 <param name="maxErrors" value="50"/>
@@
 </autorouter>
 <elements>
-<element name="LEVELSHIFTER" library="SparkFun-Boards" library_urn="urn:adsk.eagle:library:509" package="SPARKFUN_LOGIC_LEVEL_CONVERTER" package3d_urn="urn:adsk.eagle:package:37318/1" value="SPARKFUN_LOGIC_LEVEL_CONVERTER" x="57.15" y="66.04"/>
-<element name="JP1" library="SparkFun-Connectors" package="1X13" value="M13" x="38.1" y="76.2" rot="R270.7"/>
-<element name="C1" library="resistor" library_urn="urn:adsk.eagle:library:348" package="E2,5-6" package3d_urn="urn:adsk.eagle:package:25832/1" value="10uF" x="69.85" y="48.26" rot="R270.4"/>
-<element name="C2" library="resistor" library_urn="urn:adsk.eagle:library:348" package="E2,5-6" package3d_urn="urn:adsk.eagle:package:25832/1" value="10uF" x="46.99" y="46.99" rot="R270"/>
-<element name="LSM" library="pinhead" library_urn="urn:adsk.eagle:library:325" package="1X06" package3d_urn="urn:adsk.eagle:package:22472/2" value="" x="72.39" y="64.77" rot="R90"/>
-<element name="LM1117" library="pinhead" library_urn="urn:adsk.eagle:library:325" package="1X03" package3d_urn="urn:adsk.eagle:package:22458/2" value="" x="57.15" y="50.8"/>
+<element name="LEVELSHIFTER" library="SparkFun-Boards" library_urn="urn:adsk.eagle:library:509" package="SPARKFUN_LOGIC_LEVEL_CONVERTER" package3d_urn="urn:adsk.eagle:package:37318/1" value="SPARKFUN_LOGIC_LEVEL_CONVERTER" x="57.15" y="66.04" smashed="yes">
+<attribute name="NAME" x="57.15" y="73.914" size="0.6096" layer="25" font="vector" ratio="20" align="bottom-center"/>
+<attribute name="VALUE" x="57.15" y="58.166" size="0.6096" layer="25" font="vector" ratio="20" align="top-center"/>
+</element>
+<element name="JP1" library="SparkFun-Connectors" package="1X13" value="M13" x="38.1" y="76.2" smashed="yes" rot="R270.7">
+<attribute name="NAME" x="39.912215625" y="77.568440625" size="1.27" layer="25" ratio="10" rot="R270.7"/>
+<attribute name="VALUE" x="34.90971875" y="77.431115625" size="1.27" layer="27" rot="R270.7"/>
+</element>
+<element name="C1" library="resistor" library_urn="urn:adsk.eagle:library:348" package="E2,5-6" package3d_urn="urn:adsk.eagle:package:25832/1" value="10uF" x="69.85" y="48.26" smashed="yes" rot="R270.4">
+<attribute name="NAME" x="71.39258125" y="45.603703125" size="1.27" layer="25" ratio="10" rot="R270.4"/>
+<attribute name="VALUE" x="67.20168125" y="45.57444375" size="1.27" layer="27" ratio="10" rot="R270.4"/>
+</element>
+<element name="C2" library="resistor" library_urn="urn:adsk.eagle:library:348" package="E2,5-6" package3d_urn="urn:adsk.eagle:package:25832/1" value="10uF" x="46.99" y="46.99" smashed="yes" rot="R270">
+<attribute name="NAME" x="48.514" y="44.323" size="1.27" layer="25" ratio="10" rot="R270"/>
+<attribute name="VALUE" x="44.323" y="44.323" size="1.27" layer="27" ratio="10" rot="R270"/>
+</element>
+<element name="LSM" library="pinhead" library_urn="urn:adsk.eagle:library:325" package="1X06" package3d_urn="urn:adsk.eagle:package:22472/2" value="" x="72.39" y="64.77" smashed="yes" rot="R90">
+<attribute name="NAME" x="70.5612" y="57.0738" size="1.27" layer="25" ratio="10" rot="R90"/>
+<attribute name="VALUE" x="75.565" y="57.15" size="1.27" layer="27" rot="R90"/>
+</element>
+<element name="LM1117" library="pinhead" library_urn="urn:adsk.eagle:library:325" package="1X03" package3d_urn="urn:adsk.eagle:package:22458/2" value="" x="57.15" y="50.8" smashed="yes">
+<attribute name="NAME" x="53.2638" y="52.6288" size="1.27" layer="25" ratio="10"/>
+<attribute name="VALUE" x="53.34" y="47.625" size="1.27" layer="27"/>
+</element>
 </elements>
 <signals>
@@
 </signal>
 </signals>
+<mfgpreviewcolors>
+<mfgpreviewcolor name="soldermaskcolor" color="0xC8008000"/>
+<mfgpreviewcolor name="silkscreencolor" color="0xFFFEFEFE"/>
+<mfgpreviewcolor name="backgroundcolor" color="0xFF282828"/>
+<mfgpreviewcolor name="coppercolor" color="0xFFFFBF00"/>
+<mfgpreviewcolor name="substratecolor" color="0xFF786E46"/>
+</mfgpreviewcolors>
 </board>
 </drawing>
