File: Repo_PCB/final/manual_arduino_new/mega pinout.brd (EAGLE design)
At the start: 206 x 112.2 mm, 22 parts

Commit message: manual
Parts:
- turned JP2 to 90 degrees
Connections:
- removed net 32: JP1.13, JP2.2
- removed net 34: JP1.15, JP2.3
- new net N$2: JP1.15, JP2.2
- new net N$3: JP1.13, JP2.3
Routing:
- net N$2: track 0.00 -> 9.66 mm
- net 34: track 9.66 -> 0.00 mm
- net N$3: track 0.00 -> 9.66 mm
- net 32: track 9.66 -> 0.00 mm
- net GND: track 102.7 -> 96.5 mm
